File: board/board.kicad_pcb (KiCad board)
At the start: 2 copper layers, 21 x 13 mm, 1 part

Commit message: initial
Parts:
- added C1: 100nF, Capacitor_SMD:C_0402_1005Metric, F.Cu at (151.5, 94.0)
- added J1: 001_I2C, on_edge:on_edge_2x05_device, F.Cu at (140.0, 96.5)
- added J2: 001_I2C, on_edge:on_edge_2x05_host, F.Cu at (161.0, 96.5)
- added U1: STS4X, b133:STS4X, F.Cu at (149.7, 94.0)
- moved LOGO1 0.71 mm to (150.4, 99.5)
Routing:
- net /sts_40_temp/VDD: track 0.00 -> 22.1 mm, vias 0 -> 1
- net Net-(J1-Pad8): track 0.00 -> 19.6 mm
- net GND: track 0.00 -> 18.4 mm, vias 0 -> 25
- net /sts_40_temp/SCL: track 0.00 -> 18.2 mm
- net /sts_40_temp/SDA: track 0.00 -> 18.1 mm
- net Net-(J1-Pad5): track 0.00 -> 17.1 mm
- net Net-(J1-Pad10): track 0.00 -> 16.9 mm
- net Net-(J1-Pad4): track 0.00 -> 16.3 mm
- added copper zone on B.Cu, net GND
- added copper zone on F.Cu, net GND
Other:
- outline, holes or cut-outs redrawn
- board text added: "osf.001"
- board text added: "osf.b133.v1.0"
